File: Supply.sch (KiCad schematic (older format))
At the start: 10 parts, among them J501 6.5V-12V, J502 5V, U501 AZ1117-5.0

Commit message: Little interface changing.
Parts:
- D502: symbol LED -> LED-RESCUE-masterbox
Changed lines of the file:
@@
 EESchema Schematic File Version 2
+LIBS:masterbox-rescue
+LIBS:ledbox-rescue
 LIBS:power
 LIBS:device
@@
 LIBS:ledbox-newsymbols
 LIBS:switches
-LIBS:ledbox-cache
+LIBS:masterbox-cache
 EELAYER 25 0
 EELAYER END
@@
 $EndComp
 $Comp
-L +12V #PWR501
+L +12V #PWR043
 U 1 1 59DBA13C
 P 4300 3700
-F 0 "#PWR501" H 4300 3550 50  0001 C CNN
+F 0 "#PWR043" H 4300 3550 50  0001 C CNN
 F 1 "+12V" H 4300 3840 50  0000 C CNN
 F 2 "" H 4300 3700 50  0001 C CNN
@@
 $EndComp
 $Comp
-L GND #PWR502
+L GND #PWR044
 U 1 1 59DBA1A9
 P 4300 4000
-F 0 "#PWR502" H 4300 3750 50  0001 C CNN
+F 0 "#PWR044" H 4300 3750 50  0001 C CNN
 F 1 "GND" H 4300 3850 50  0000 C CNN
 F 2 "" H 4300 4000 50  0001 C CNN
@@
 $EndComp
 $Comp
-L GND #PWR504
+L GND #PWR045
 U 1 1 59DBA33D
 P 4300 4700
-F 0 "#PWR504" H 4300 4450 50  0001 C CNN
+F 0 "#PWR045" H 4300 4450 50  0001 C CNN
 F 1 "GND" H 4300 4550 50  0000 C CNN
 F 2 "" H 4300 4700 50  0001 C CNN
@@
 $EndComp
 $Comp
-L +5V #PWR503
+L +5V #PWR046
 U 1 1 59DBA35E
 P 4300 4400
-F 0 "#PWR503" H 4300 4250 50  0001 C CNN
+F 0 "#PWR046" H 4300 4250 50  0001 C CNN
 F 1 "+5V" H 4300 4540 50  0000 C CNN
 F 2 "" H 4300 4400 50  0001 C CNN
@@
 $EndComp
 $Comp
-L +12V #PWR505
+L +12V #PWR047
 U 1 1 59DBA74B
 P 5100 3900
-F 0 "#PWR505" H 5100 3750 50  0001 C CNN
+F 0 "#PWR047" H 5100 3750 50  0001 C CNN
 F 1 "+12V" H 5100 4040 50  0000 C CNN
 F 2 "" H 5100 3900 50  0001 C CNN
@@
 $EndComp
 $Comp
-L GND #PWR506
+L GND #PWR048
 U 1 1 59DBA861
 P 5800 4600
-F 0 "#PWR506" H 5800 4350 50  0001 C CNN
+F 0 "#PWR048" H 5800 4350 50  0001 C CNN
 F 1 "GND" H 5800 4450 50  0000 C CNN
 F 2 "" H 5800 4600 50  0001 C CNN
@@
 $EndComp
 $Comp
-L +5V #PWR507
+L +5V #PWR049
 U 1 1 59DBAA1E
 P 6500 3900
-F 0 "#PWR507" H 6500 3750 50  0001 C CNN
+F 0 "#PWR049" H 6500 3750 50  0001 C CNN
 F 1 "+5V" H 6500 4040 50  0000 C CNN
 F 2 "" H 6500 3900 50  0001 C CNN
@@
 	5650 3700 5400 3700
 $Comp
-L LED D502
+L LED-RESCUE-masterbox D502
 U 1 1 59E32AE2
 P 7100 4050
+AR Path="/59E32AE2" Ref="D502"  Part="1"
+AR Path="/59DBA013/59E32AE2" Ref="D502"  Part="1"
 F 0 "D502" H 7100 4150 50  0000 C CNN
 F 1 "LED2" H 7100 3950 50  0000 C CNN
@@
 $EndComp
 $Comp
-L +5V #PWR508
+L +5V #PWR050
 U 1 1 59E32AF0
 P 7100 3800
-F 0 "#PWR508" H 7100 3650 50  0001 C CNN
+F 0 "#PWR050" H 7100 3650 50  0001 C CNN
 F 1 "+5V" H 7100 3940 50  0000 C CNN
 F 2 "" H 7100 3800 50  0001 C CNN
@@
 	7100 4200 7100 4300
 $Comp
-L GND #PWR509
+L GND #PWR051
 U 1 1 59E32B42
 P 7100 4700
-F 0 "#PWR509" H 7100 4450 50  0001 C CNN
+F 0 "#PWR051" H 7100 4450 50  0001 C CNN
 F 1 "GND" H 7100 4550 50  0000 C CNN
 F 2 "" H 7100 4700 50  0001 C CNN
