File: Bus.sch (KiCad schematic (older format))
At the start: 15 parts, among them J201 Bus, U201 ST485C

Commit message: ATmega2560 inserted
Changed lines of the file:
@@
 	7000 4800 7000 4500
 Wire Wire Line
-	6900 4500 7100 4500
-Wire Wire Line
-	8500 5100 8900 5100
-Wire Wire Line
-	8500 5000 8500 5200
+	6900 4500 7000 4500
+Wire Wire Line
+	7000 4500 7100 4500
+Wire Wire Line
+	8500 5100 8800 5100
+Wire Wire Line
+	8800 5100 8900 5100
+Wire Wire Line
+	8500 5000 8500 5100
+Wire Wire Line
+	8500 5100 8500 5200
 Connection ~ 8500 5100
 Wire Wire Line
@@
 	8800 5200 8800 5100
 Wire Wire Line
-	7400 4500 7900 4500
+	7400 4500 7500 4500
+Wire Wire Line
+	7500 4500 7800 4500
+Wire Wire Line
+	7800 4500 7900 4500
 Connection ~ 7000 4500
 Wire Wire Line
@@
 	1500 3400 1900 3400
 Wire Wire Line
-	2900 3400 3700 3400
-Wire Wire Line
-	3100 3300 3100 3450
-Wire Wire Line
-	2900 3800 3700 3800
-Wire Wire Line
-	3100 3750 3100 3900
+	2900 3400 3100 3400
+Wire Wire Line
+	3100 3400 3700 3400
+Wire Wire Line
+	3100 3300 3100 3400
+Wire Wire Line
+	3100 3400 3100 3450
+Wire Wire Line
+	2900 3800 3100 3800
+Wire Wire Line
+	3100 3800 3700 3800
+Wire Wire Line
+	3100 3750 3100 3800
+Wire Wire Line
+	3100 3800 3100 3900
 Connection ~ 3100 3800
 Connection ~ 3100 3400
@@
 	7750 3350 7650 3350
 Wire Wire Line
-	7650 3250 7650 3450
+	7650 3250 7650 3350
+Wire Wire Line
+	7650 3350 7650 3450
 Wire Wire Line
 	7650 3450 7750 3450
 Connection ~ 7650 3350
 Wire Wire Line
-	8250 3350 8450 3350
+	8250 3350 8350 3350
+Wire Wire Line
+	8350 3350 8450 3350
 Wire Wire Line
 	8350 3350 8350 3450
@@
 Connection ~ 8350 3350
 Wire Wire Line
-	8250 3650 8450 3650
+	8250 3650 8350 3650
+Wire Wire Line
+	8350 3650 8450 3650
 Wire Wire Line
 	8250 3750 8350 3750
@@
 Connection ~ 8350 3650
 Wire Wire Line
-	7650 3650 7650 3850
+	7650 3650 7650 3750
+Wire Wire Line
+	7650 3750 7650 3850
 Wire Wire Line
 	7650 3650 7750 3650
